Commit message: add missing resources for gazebo

File: active_perception_evaluation/urdf/race_coffee_cup_hot.urdf.xacro (robot description, xacro)
@@ -1,5 +1,5 @@
 <robot
   xmlns:xacro="http://ros.org/wiki/xacro"
-  name="race_mug3">
+  name="race_mug_hot">
   <include filename="$(find active_perception_evaluation)/urdf/common.xacro" />
   <xacro:property name="cup_radius" value="0.04" />
@@ -25,5 +25,5 @@
   </link>
   <gazebo reference="body">
-    <material>Gazebo/WhiteGlow</material>
+    <material>Gazebo/RedGlow</material>
   </gazebo>
 </robot>
